File: eurobot2023/Electronics/main_pcb/main_pcb.kicad_pcb (KiCad board)
At the start: 2 copper layers, 120.9 x 93.2 mm, 37 parts, among them IC1 74HCT541D,652, IC2 SN74LVC126ADR, IC3 74HCT1G125GW, J1 PI40HAT, J10 Conn_01x02_Male, J11 MagneticEncoder, J12 Conn_01x07_Male, J13 MagneticEncoder, J14 Conn_01x03_Male, J15 Conn_01x02_Male, J2 Conn_01x02_Male, J3 Conn_01x02_Male, J4 Conn_01x02_Male, J5 Conn_01x02_Male, J6 Conn_01x02_Male, J7 Conn_01x02_Male, J9 22-03-5035, P1 R-78Bxx-2.0, P2 Amazon 10A stepdown, U1 MCP2515-xSO, U2 TJA1049T, U3 PCA9306D, U4 Pololu_MAX14870, U5 PCA9685PW

Commit message: Update serigraphies
Parts:
- moved R2 52.8 mm to (141.0, 132.1)
- moved R4 13.4 mm to (79.4, 62.2), turned to 180 degrees
- moved U4 6.20 mm to (170.8, 96.5)
- moved C3 5.28 mm to (180.8, 90.8)
- moved J10 4.71 mm to (179.7, 115.6)
- moved C4 4.21 mm to (68.6, 101.6)
- moved J14 3.28 mm to (129.6, 90.2)
- moved J6 1.55 mm to (173.4, 142.8)
- moved J15 1.54 mm to (179.6, 125.0)
- moved J5 1.36 mm to (74.9, 140.9)
- moved J9 1.27 mm to (181.0, 59.0)
- moved J7 0.45 mm to (68.6, 123.2)
- moved J12 0.19 mm to (68.6, 73.0)
Other:
- board text added: "0"
- board text added: "1"
- board text added: "2"
- board text added: "20"
- board text added: "21"
- board text added: "22"
- board text added: "23"
- board text added: "3"
- board text added: "3V3"
- board text added: "4"
- board text added: "5"
- board text added: "5V"
- board text added: "6"
- board text added: "7"
- board text added: "7V5"
- board text added: "A0"
- board text added: "CANH"
- board text added: "CANL"
- board text added: "GND"
- board text added: "GPIO"
- board text added: "I2C SCL"
- board text added: "I2C SDA"
- board text added: "M1"
- board text added: "M2"
- board text added: "UART RX"
