File: Electronics/esp32-powerswitcher/esp32-powerswitcher.kicad_pcb (KiCad board)
At the start: 2 copper layers, 38 x 43 mm, 50 parts, among them J1 Conn_01x04_Male, J2 Conn_01x04_Male, J3 Conn_01x02_Male, J4 Conn_01x02_Male, J5 Conn_01x03_Pin, Q1 NVTR4503NT1G, Q2 NVTR4503NT1G, Q3 NVTR4503NT1G, Q4 NVTR4503NT1G, Q5 NVTR4503NT1G, Q6 NVTR4503NT1G, Q7 NVTR4503NT1G, Q8 NVTR4503NT1G, U1 MODULE-SEEEDUINO-XIAO-ESP32C3

Commit message: PCB fixup
Parts:
- added IC1: TCA9416DDFR, MiAM:SOT65P280X110-8N, F.Cu at (114.4, 74.8)
- added J6: Conn_01x04_Male, Connector_JST:JST_SH_SM04B-SRSS-TB_1x04-1MP_P1.00mm_Horizontal, F.Cu at (118.8, 64.4)
- added JP1: SolderJumper_2_Open, Jumper:SolderJumper-2_P1.3mm_Open_Pad1.0x1.5mm, F.Cu at (109.2, 70.2)
- added R11: 4.7k, Resistor_SMD:R_0805_2012Metric_Pad1.20x1.40mm_HandSolder, F.Cu at (115.2, 69.7)
- added R12: 4.7k, Resistor_SMD:R_0805_2012Metric_Pad1.20x1.40mm_HandSolder, F.Cu at (117.1, 69.7)
- moved R3 3.41 mm to (119.9, 68.8)
- moved R4 2.81 mm to (119.9, 70.7)
- moved R2 2.22 mm to (112.4, 68.6), turned to 180 degrees
- moved R5 2.11 mm to (119.5, 72.6)
- moved J2 1.81 mm to (111.0, 64.4)
- moved R6 1.51 mm to (119.5, 74.5)
- moved R1 1.14 mm to (112.4, 70.5), turned to 180 degrees
- moved R10 1.10 mm to (110.2, 74.1)
- moved R9 0.50 mm to (110.2, 76.0)
- moved D8 0.37 mm to (101.4, 72.2)
- moved R8 0.30 mm to (110.2, 78.4)
- moved D7 0.10 mm to (101.4, 79.1)
Connections:
- net Net-(J5-Pin_1) renamed /S6
- R1 pad 1: +3.3V -> /I2C3.3
- R2 pad 1: +3.3V -> /I2C3.3
Routing:
- net /I2C3.3: track 35.7 -> 13.8 mm, vias 2 -> 0
- net Net-(IC1-SDA_B): track 0.00 -> 8.91 mm, vias 0 -> 2
- net Net-(IC1-SCL_B): track 0.00 -> 8.23 mm, vias 0 -> 2
- net /S6: track 20.6 -> 27.6 mm, vias 1 -> 3
- net +3.3V: track 5.10 -> 2.46 mm
- net /SCL: track 47.7 -> 45.5 mm, vias 1 -> 4
- net /SDA: track 47.6 -> 49.6 mm, vias 0 -> 3
- net GND: track 29.7 -> 30.9 mm, vias 24 -> 23
- net /S1: track 12.1 -> 13.2 mm
- net /S2: track 16.2 -> 17.0 mm
- net /S7: track 13.1 -> 12.5 mm
- added copper zone on F.Cu, net /I2C3.3
Other:
- board text added: "3.3V"
- board text added: "I2C AUX"
