File: Electronics/esp32-powerswitcher/esp32-powerswitcher.kicad_sch (KiCad schematic)
At the start: 50 parts, among them J1 Conn_01x04_Male, J2 Conn_01x04_Male, J3 Conn_01x02_Male, J4 Conn_01x02_Male, J5 Conn_01x03_Pin, Q1 NVTR4503NT1G, Q2 NVTR4503NT1G, Q3 NVTR4503NT1G, Q4 NVTR4503NT1G, Q5 NVTR4503NT1G, Q6 NVTR4503NT1G, Q7 NVTR4503NT1G, Q8 NVTR4503NT1G, U1 MODULE-SEEEDUINO-XIAO-ESP32C3

Commit message: PCB fixup
Parts:
- added IC1: TCA9416DDFR, MiAM:SOT65P280X110-8N, symbol MiAM:TCA9416DDFR
- added J6: Conn_01x04_Male, Connector_JST:JST_SH_SM04B-SRSS-TB_1x04-1MP_P1.00mm_Horizontal, symbol Connector:Conn_01x04_Male
- added JP1: SolderJumper_2_Open, Jumper:SolderJumper-2_P1.3mm_Open_Pad1.0x1.5mm, symbol Jumper:SolderJumper_2_Open
- added R11, R12: 4.7k, Resistor_SMD:R_0805_2012Metric_Pad1.20x1.40mm_HandSolder, symbol Device:R
Connections:
- net +3.3V: now also JP1.2 (B); no longer R1.1, R2.1
- net GND: now also J6.1 (Pin_1)
- net I2C3.3: now also R1.1, R2.1, IC1.3 (VCCA), IC1.7 (VCCB), J6.2 (Pin_2), JP1.1 (A), R11.1, R12.1
- net SCL: now also IC1.1 (SCL_A)
- net SDA: now also IC1.4 (SDA_A)
- net S6: now reaches J5.1 (Pin_1), U1.7 (PB08_A6_D6_TX)
- net S6: now also IC1.2 (OE)
- new net: IC1.5 (SDA_B), J6.3 (Pin_3), R12.2
- new net: IC1.8 (SCL_B), J6.4 (Pin_4), R11.2
Other:
- moved on the sheet: J1
