File: Electronics/main_pcb_2026/main_pcb_2026.kicad_pcb (KiCad board)
At the start: 4 copper layers, 56 x 65.5 mm, 57 parts, among them IC2 PCA9543AD,118, J1 PI40HAT, J10 Conn_01x03_Pin, J14 Conn_01x02_Pin, J2 MilliMax0600, J23 22-03-5035, J28 MilliMax0600, J29 MilliMax0600, J3 MilliMax0600, J30 MilliMax0600, J31 22-03-5035, J32 22-03-5035, J4 MilliMax0600, J5 Conn_01x02_Male, J6 Conn_01x02_Male, J7 217175-0001, J8 Conn_01x02_Male, J9 22-03-5035, U1 SN74AHCT1G126DBVR, U3 R-78B5.0-2.0, U4 Pololu_MAX14870, U5 SN74LVC1G125DBVR, U6 Pololu_MAX14870

Commit message: PCB fixup
Parts:
- R5: value 4k -> 20k
- moved R11 2.80 mm to (127.7, 65.5)
- moved R12 2.80 mm to (125.7, 65.5)
- moved I2C1 2.51 mm to (127.5, 60.5)
- moved R6 2.28 mm to (90.3, 60.3)
- moved R1 2.27 mm to (90.3, 62.3)
- moved I2C4 2.00 mm to (96.3, 60.4)
- moved R15 1.00 mm to (107.4, 65.5)
- moved R16 1.00 mm to (105.4, 65.5)
- moved I2C2 0.49 mm to (106.7, 60.3)
- moved R17 0.12 mm to (90.1, 82.0)
- moved I2C0 0.10 mm to (117.1, 60.3)
Routing:
- net Net-(IC2-~{INT}): track 8.58 -> 12.6 mm
- net +24V: track 8.96 -> 6.01 mm
- net /SDA1: track 33.9 -> 35.2 mm
- net /SCL1: track 29.3 -> 30.5 mm
- net /I2C SDA: track 75.8 -> 76.6 mm
- net /GPIO 19: track 26.5 -> 25.9 mm
- net GND: track 19.2 -> 18.9 mm, vias 85 -> 298
- removed copper zone on F.Cu, net GND
