File: Electronics/main_pcb_2026/main_pcb_2026.kicad_sch (KiCad schematic)
At the start: 57 parts, among them IC2 PCA9543AD,118, J1 PI40HAT, J10 Conn_01x03_Pin, J14 Conn_01x02_Pin, J2 MilliMax0600, J23 22-03-5035, J28 MilliMax0600, J29 MilliMax0600, J3 MilliMax0600, J30 MilliMax0600, J31 22-03-5035, J32 22-03-5035, J4 MilliMax0600, J5 Conn_01x02_Male, J6 Conn_01x02_Male, J7 217175-0001, J8 Conn_01x02_Male, J9 22-03-5035, U1 SN74AHCT1G126DBVR, U3 R-78B5.0-2.0, U4 Pololu_MAX14870, U5 SN74LVC1G125DBVR, U6 Pololu_MAX14870

Commit message: PCB fixup
Parts:
- R5: value 4k -> 20k
Changed lines of the file:
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@@
 			)
 		)
-		(property "Value" "4k"
+		(property "Value" "20k"
 			(at 317.5 48.2599 0)
 			(effects
