File: Electronics/power_supply/power_supply.kicad_sch (KiCad schematic)
At the start: 83 parts, among them IC1 TLV76033DBZR, IC2 LM5069MMX-2_NOPB, J1 Conn_01x02_Male, J10 9801-0-15-15-23-27-10-0, J12 9801-0-15-15-23-27-10-0, J13 9801-0-15-15-23-27-10-0, J14 9801-0-15-15-23-27-10-0, J2 9801-0-15-15-23-27-10-0, J3 Conn_01x02_Male, J4 821-22-002-10-001101, J5 9801-0-15-15-23-27-10-0, J6 Conn_01x04_Male, J7 Conn_01x02_Male, J8 Conn_01x02_Male, J9 Conn_01x02_Pin, Q1 IPD90N04S4L04ATMA1, Q3 MMBT5401, U1 R-78B5.0-2.0, U2 INA226, U3 INA226

Commit message: PCB fixup
Parts:
- J4: now fitted
Changed lines of the file:
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@@
 		(in_bom yes)
 		(on_board yes)
-		(dnp yes)
+		(dnp no)
 		(fields_autoplaced yes)
 		(property "Reference" "J4"
